File: HyperFuzz.kicad_sch (KiCad schematic)
At the start: 62 parts, among them J1 9V, J2 G, J3 IN/LED/GND/OUT, J4 IG, J5 OG, U1 TL072, U2 TL072, U3 TL072

Commit message: Hyper Fuzz v1.1: 9 mm pots, new knob grid, wire pads moved, enclosure drilling
As ordered from JLCPCB (October 2026 batch).

Co-Authored-By: Claude Opus 5.5 <noreply@anthropic.com>
Parts:
- added C12: 1n, Capacitor_SMD:C_0805_2012Metric_Pad1.18x1.45mm_HandSolder, symbol Device:C
- added C13: 100p, Capacitor_SMD:C_0805_2012Metric_Pad1.18x1.45mm_HandSolder, symbol Device:C
- added R27: 1M, Resistor_SMD:R_0805_2012Metric_Pad1.20x1.40mm_HandSolder, symbol Device:R
- RV1, RV2, RV3, RV4, RV5: footprint UglyFace:Potentiometer_Alpha_16mm_Vertical -> Potentiometer_THT:Potentiometer_Alpha_RD901F-40-00D_Single_Vertical
- U3: value TL072 -> LM358; LCSC C6961 -> C7950
Connections:
- net GND: now also C12.2, R27.2
- net IN: now also R27.1
- net PRE: now also C13.2
- net at R3.1, R4.1, U1.2 (-): now also C13.1
- net at C1.1, R1.2: now also C12.1
Other:
- moved on the sheet: C1, C2, C4, C5, D10, D3, D4, D5, D6, D7, D8, D9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
